Commit message: use end stops for zero pos (#30)
* read end stops

* zero pos script

---------

Co-authored-by: Almond Workstation <workstation@almondbot.com>

File: almond_axol/kinematics/urdf/axol.urdf (robot description, URDF)
Before this commit: robot assembly, 19 links, 18 joints
Joints:
- joint left_e1_0: limit lower=0.0 upper=2.6389 effort=87.0 velocity=30.0 -> lower=0.0 upper=2.6180 effort=87.0 velocity=30.0
- joint left_e2_0: limit lower=-1.5708 upper=1.5708 effort=87.0 velocity=30.0 -> lower=-2.3562 upper=2.3562 effort=87.0 velocity=30.0
- joint left_s1_0: limit lower=-1.5708 upper=1.5708 effort=87.0 velocity=30.0 -> lower=-1.5708 upper=3.1416 effort=87.0 velocity=30.0
- joint left_s2_0: limit lower=-1.5708 upper=0.1885 effort=87.0 velocity=30.0 -> lower=-3.1416 upper=0.3491 effort=87.0 velocity=30.0
- joint left_s3_0: limit lower=-1.5708 upper=1.5708 effort=87.0 velocity=30.0 -> lower=-2.3562 upper=2.3562 effort=87.0 velocity=30.0
- joint right_e1_0: limit lower=-2.6389 upper=0.0 effort=87.0 velocity=30.0 -> lower=-2.6180 upper=0.0 effort=87.0 velocity=30.0
- joint right_e2_0: limit lower=-1.5708 upper=1.5708 effort=87.0 velocity=30.0 -> lower=-2.3562 upper=2.3562 effort=87.0 velocity=30.0
- joint right_s1_0: limit lower=-1.5708 upper=1.5708 effort=87.0 velocity=30.0 -> lower=-3.1416 upper=1.5708 effort=87.0 velocity=30.0
- joint right_s2_0: limit lower=-0.1885 upper=1.5708 effort=87.0 velocity=30.0 -> lower=-0.3491 upper=3.1416 effort=87.0 velocity=30.0
- joint right_s3_0: limit lower=-1.5708 upper=1.5708 effort=87.0 velocity=30.0 -> lower=-2.3562 upper=2.3562 effort=87.0 velocity=30.0
